File: L6235.sch (KiCad schematic (older format))
At the start: 28 parts, among them P1 CONN_01X03, U1 L6235N

Commit message: fix: larger GND plan next to Phase2
Changed lines of the file:
@@
 LIBS:motor_drivers
 LIBS:motor_drivers_custom
-LIBS:L6235-cache
 EELAYER 25 0
 EELAYER END
@@
 L PWR_FLAG #FLG012
 U 1 1 577FA886
-P 2350 5900
-F 0 "#FLG012" H 2350 5995 50  0001 C CNN
-F 1 "PWR_FLAG" H 2350 6080 50  0000 C CNN
-F 2 "" H 2350 5900 50  0000 C CNN
-F 3 "" H 2350 5900 50  0000 C CNN
-	1    2350 5900
+P 2500 6300
+F 0 "#FLG012" H 2500 6395 50  0001 C CNN
+F 1 "PWR_FLAG" H 2500 6480 50  0000 C CNN
+F 2 "" H 2500 6300 50  0000 C CNN
+F 3 "" H 2500 6300 50  0000 C CNN
+	1    2500 6300
 	1    0    0    -1
 $EndComp
@@
 L PWR_FLAG #FLG013
 U 1 1 577FA8EF
-P 2750 5900
-F 0 "#FLG013" H 2750 5995 50  0001 C CNN
-F 1 "PWR_FLAG" H 2750 6080 50  0000 C CNN
-F 2 "" H 2750 5900 50  0000 C CNN
-F 3 "" H 2750 5900 50  0000 C CNN
-	1    2750 5900
+P 2900 6300
+F 0 "#FLG013" H 2900 6395 50  0001 C CNN
+F 1 "PWR_FLAG" H 2900 6480 50  0000 C CNN
+F 2 "" H 2900 6300 50  0000 C CNN
+F 3 "" H 2900 6300 50  0000 C CNN
+	1    2900 6300
 	1    0    0    -1
 $EndComp
@@
 L PWR_FLAG #FLG014
 U 1 1 577FA951
-P 3150 5900
-F 0 "#FLG014" H 3150 5995 50  0001 C CNN
-F 1 "PWR_FLAG" H 3150 6080 50  0000 C CNN
-F 2 "" H 3150 5900 50  0000 C CNN
-F 3 "" H 3150 5900 50  0000 C CNN
-	1    3150 5900
+P 3300 6300
+F 0 "#FLG014" H 3300 6395 50  0001 C CNN
+F 1 "PWR_FLAG" H 3300 6480 50  0000 C CNN
+F 2 "" H 3300 6300 50  0000 C CNN
+F 3 "" H 3300 6300 50  0000 C CNN
+	1    3300 6300
 	1    0    0    -1
 $EndComp
@@
 L GND #PWR015
 U 1 1 577FA998
-P 2350 6000
-F 0 "#PWR015" H 2350 5750 50  0001 C CNN
-F 1 "GND" H 2350 5850 50  0000 C CNN
-F 2 "" H 2350 6000 50  0000 C CNN
-F 3 "" H 2350 6000 50  0000 C CNN
-	1    2350 6000
+P 2500 6400
+F 0 "#PWR015" H 2500 6150 50  0001 C CNN
+F 1 "GND" H 2500 6250 50  0000 C CNN
+F 2 "" H 2500 6400 50  0000 C CNN
+F 3 "" H 2500 6400 50  0000 C CNN
+	1    2500 6400
 	1    0    0    -1
 $EndComp
@@
 L +5V #PWR016
 U 1 1 577FAB36
-P 2750 6000
-F 0 "#PWR016" H 2750 5850 50  0001 C CNN
-F 1 "+5V" H 2750 6140 50  0000 C CNN
-F 2 "" H 2750 6000 50  0000 C CNN
-F 3 "" H 2750 6000 50  0000 C CNN
-	1    2750 6000
+P 2900 6400
+F 0 "#PWR016" H 2900 6250 50  0001 C CNN
+F 1 "+5V" H 2900 6540 50  0000 C CNN
+F 2 "" H 2900 6400 50  0000 C CNN
+F 3 "" H 2900 6400 50  0000 C CNN
+	1    2900 6400
 	-1   0    0    1
 $EndComp
@@
 L VSS #PWR017
 U 1 1 577FAD9E
-P 3150 6000
-F 0 "#PWR017" H 3150 5850 50  0001 C CNN
-F 1 "VSS" H 3150 6150 50  0000 C CNN
-F 2 "" H 3150 6000 50  0000 C CNN
-F 3 "" H 3150 6000 50  0000 C CNN
-	1    3150 6000
+P 3300 6400
+F 0 "#PWR017" H 3300 6250 50  0001 C CNN
+F 1 "VSS" H 3300 6550 50  0000 C CNN
+F 2 "" H 3300 6400 50  0000 C CNN
+F 3 "" H 3300 6400 50  0000 C CNN
+	1    3300 6400
 	-1   0    0    1
 $EndComp
@@
 	2750 2450 3150 2450
 Wire Wire Line
-	2350 5900 2350 6000
-Wire Wire Line
-	2750 5900 2750 6000
-Wire Wire Line
-	3150 5900 3150 6000
+	2500 6300 2500 6400
+Wire Wire Line
+	2900 6300 2900 6400
+Wire Wire Line
+	3300 6300 3300 6400
 Wire Wire Line
 	3450 3600 2400 3600
